Commit message: fix: controller spawning; removed robotNamespace argument in gazebo plugin implementation in iiwa.gazebo.xacro causing confliction and controller to not be spawning with expected name; controllers yaml file to be more consistent with other armada/forked robot packages, TODO: explore robotNamespace argument further; intended use and functionality to add more namespace flexibility to project

File: iiwa_description/grippers/robotiq_2f_140/urdf/robotiq_2f_140_transmission_macro.xacro (robot description, xacro)
@@ -55,6 +55,6 @@
             <plugin name="gazebo_grasp_fix" filename="libgazebo_grasp_fix.so">
                 <arm>
-                    <arm_name>ur5e</arm_name>
-                    <palm_link>${prefix}iiwa7_link_ee</palm_link>
+                    <arm_name>iiwa7</arm_name>
+                    <palm_link>${prefix}iiwa_link_7</palm_link>
                     <!-- Gazebo merges links connected by fixed joints, so you need to check the links in gazebo and choose one that is recognized after internal connections are made. We would want to choose the actual paml of the gripper but it is currently not an option THIS VALUE WILL NEED TO CHANGE FOR THE IIWA14 WHICH IS NOT CURRENTLY BEING USED; A VARIABLE SUCH AS "MODEL" SHOULD BE PASSED IN IN THIS CASE-->
                     <gripper_link> ${prefix}left_inner_finger </gripper_link>

File: iiwa_description/grippers/robotiq_2f_85/urdf/robotiq_2f_85_transmission_macro.xacro (robot description, xacro)
@@ -56,5 +56,5 @@
                 <arm>
                     <arm_name>iiwa7</arm_name>
-                    <palm_link>${prefix}iiwa7_link_ee</palm_link>
+                    <palm_link>${prefix}iiwa_link_7</palm_link>
                     <!-- Gazebo merges links connected by fixed joints, so you need to check the links in gazebo and choose one that is recognized after internal connections are made. We would want to choose the actual paml of the gripper but it is currently not an option THIS VALUE WILL NEED TO CHANGE FOR THE IIWA14 WHICH IS NOT CURRENTLY BEING USED; A VARIABLE SUCH AS "MODEL" SHOULD BE PASSED IN IN THIS CASE-->
                     <gripper_link> ${prefix}left_inner_finger </gripper_link>

File: iiwa_description/urdf/iiwa.gazebo.xacro (robot description, xacro)
@@ -16,6 +16,6 @@
     <!-- Load Gazebo lib and set the robot namespace -->
     <gazebo>
-      <plugin name="gazebo_ros_control" filename="libgazebo_ros_control.so">
-        <robotNamespace>/${robot_name}</robotNamespace>
+      <plugin name="ros_control" filename="libgazebo_ros_control.so">
+        <!-- <robotNamespace>/${robot_name}</robotNamespace> TODO: Look into this later, the controllers do not work with this line currently, likely has to do with namespace -->
       </plugin>
     </gazebo>

File: iiwa_description/urdf/iiwa7_robotiq_2f_140.urdf.xacro (robot description, xacro)
@@ -9,5 +9,5 @@
   <xacro:include filename="$(find iiwa_description)/grippers/robotiq_2f_140/urdf/robotiq_2f_140_transmission_macro.xacro" />
   <xacro:arg name="hardware_interface" default="PositionJointInterface"/>
-  <xacro:arg name="robot_name" default="iiwa7"/>
+  <xacro:arg name="robot_name" default="iiwa"/>
   <xacro:arg name="origin_xyz" default="0 0 0"/>
   <xacro:arg name="origin_rpy" default="0 0 0"/>

File: iiwa_description/urdf/iiwa7_robotiq_2f_140_workstation.urdf.xacro (robot description, xacro)
@@ -11,5 +11,5 @@
   <xacro:include filename="$(find iiwa_description)/grippers/robotiq_2f_85/urdf/robotiq_2f_140_transmission_macro.xacro" />
   <xacro:arg name="hardware_interface" default="PositionJointInterface"/>
-  <xacro:arg name="robot_name" default="iiwa7"/>
+  <xacro:arg name="robot_name" default="iiwa"/>
   <xacro:arg name="origin_xyz" default="0 0 0"/>
   <xacro:arg name="origin_rpy" default="0 0 0"/>
@@ -21,11 +21,6 @@
     <origin xyz="0.0 0.0 0.41" rpy="0.0 0.0 0.0" />
   </joint>
-  <joint name="connect_table_and_arm" type="fixed">
-    <parent link="table_mounting_plate_link" />
-    <child link = "$(arg robot_name)_link_0" />
-    <origin xyz="0.0 0.0 0.03625" rpy="0.0 0.0 ${pi/2}" />
-  </joint>
   <!--iiwa-->
-  <xacro:iiwa7 hardware_interface="$(arg hardware_interface)" robot_name="$(arg robot_name)" parent="world">
+  <xacro:iiwa7 hardware_interface="$(arg hardware_interface)" robot_name="$(arg robot_name)" parent="table_mounting_plate_link">
     <origin xyz="$(arg origin_xyz)" rpy="$(arg origin_rpy)" />
   </xacro:iiwa7>

File: iiwa_description/urdf/iiwa7_robotiq_2f_85_workstation.urdf.xacro (robot description, xacro)
@@ -21,11 +21,4 @@
     <origin xyz="0.0 0.0 0.41" rpy="0.0 0.0 0.0" />
   </joint>
-  <!--
-  <joint name="connect_table_and_arm" type="fixed">
-    <parent link="table_mounting_plate_link" />
-    <child link = "$(arg robot_name)_link_0" />
-    <origin xyz="0.0 0.0 0.03625" rpy="0.0 0.0 ${pi/2}" />
-  </joint>
-  -->
   <!--iiwa-->
   <xacro:iiwa7 hardware_interface="$(arg hardware_interface)" robot_name="$(arg robot_name)" parent="table_mounting_plate_link">

File: iiwa_description/urdf/iiwa7_workstation.urdf.xacro (robot description, xacro)
@@ -5,4 +5,6 @@
   <!--Import the lbr iiwa macro -->
   <xacro:include filename="$(find iiwa_description)/urdf/iiwa7.xacro"/>
+  <!-- ARMada workstation -->
+  <xacro:include filename="$(find uml_hri_nerve_armada_workstation)/workstation_description/workstation_model.urdf.xacro" />
   <xacro:arg name="hardware_interface" default="PositionJointInterface"/>
   <xacro:arg name="robot_name" default="iiwa"/>
@@ -10,8 +12,15 @@
   <xacro:arg name="origin_rpy" default="0 0 0"/>
   <!-- Fix to world just for testing -->
-  <link name="world"/>
+  <link name="world" />
+  <joint name="connect_world_and_table" type="fixed">
+    <child link="table_base_link" />
+    <parent link="world" />
+    <origin xyz="0.0 0.0 0.41" rpy="0.0 0.0 0.0" />
+  </joint>
   <!--iiwa-->
-  <xacro:iiwa7 hardware_interface="$(arg hardware_interface)" robot_name="$(arg robot_name)" parent="world">
+  <xacro:iiwa7 hardware_interface="$(arg hardware_interface)" robot_name="$(arg robot_name)" parent="table_mounting_plate_link">
     <origin xyz="$(arg origin_xyz)" rpy="$(arg origin_rpy)" />
   </xacro:iiwa7>
+  <!-- workstation -->
+  <xacro:workstation prefix="table_" namespace=""/>
 </robot>
